File: Perris_Breakout.kicad_sch (KiCad schematic)
At the start: 21 parts, among them J1 PERRI_1, J10 SDA, J11 GND, J12 GND, J13 SCL, J14 SCL, J2 PERRI_2, J3 PERRI_3, J4 PERRI_4, J5 PERRI_5, J6 PERRI_6, J7 PERRI_7, J8 PERRI_8, J9 SDA

Commit message: More Perris
Parts:
- removed J10, J9: SDA, Connector_PinHeader_2.54mm:PinHeader_1x01_P2.54mm_Vertical, symbol Connector:Conn_01x01_Male
- removed J11, J12: GND, Connector_PinHeader_2.54mm:PinHeader_1x01_P2.54mm_Vertical, symbol Connector:Conn_01x01_Male
- removed J13, J14: SCL, Connector_PinHeader_2.54mm:PinHeader_1x01_P2.54mm_Vertical, symbol Connector:Conn_01x01_Male
- removed TP1: SDA, Connector_PinHeader_2.54mm:PinHeader_1x01_P2.54mm_Vertical, symbol Connector:TestPoint_Small
- removed TP2: GND, Connector_PinHeader_2.54mm:PinHeader_1x01_P2.54mm_Vertical, symbol Connector:TestPoint_Small
- removed TP3: SCL, Connector_PinHeader_2.54mm:PinHeader_1x01_P2.54mm_Vertical, symbol Connector:TestPoint_Small
- added J10: PERRI_10, HELIX:Perri_conn_2x5_Reverse, symbol Connector_Generic:Conn_02x05_Counter_Clockwise
- added J11: PERRI_11, HELIX:Perri_conn_2x5_Reverse, symbol Connector_Generic:Conn_02x05_Counter_Clockwise
- added J12: PERRI_12, HELIX:Perri_conn_2x5_Reverse, symbol Connector_Generic:Conn_02x05_Counter_Clockwise
- added J13: PERRI_13, HELIX:Perri_conn_2x5_Reverse, symbol Connector_Generic:Conn_02x05_Counter_Clockwise
- added J14: PERRI_14, HELIX:Perri_conn_2x5_Reverse, symbol Connector_Generic:Conn_02x05_Counter_Clockwise
- added J15: PERRI_15, HELIX:Perri_conn_2x5_Reverse, symbol Connector_Generic:Conn_02x05_Counter_Clockwise
- added J16: PERRI_16, HELIX:Perri_conn_2x5_Reverse, symbol Connector_Generic:Conn_02x05_Counter_Clockwise
- added J17: PERRI_17, HELIX:Perri_conn_2x5_Reverse, symbol Connector_Generic:Conn_02x05_Counter_Clockwise
- added J18: PERRI_18, HELIX:Perri_conn_2x5_Reverse, symbol Connector_Generic:Conn_02x05_Counter_Clockwise
- added J19: PERRI_19, HELIX:Perri_conn_2x5_Reverse, symbol Connector_Generic:Conn_02x05_Counter_Clockwise
- added J20: PERRI_20, HELIX:Perri_conn_2x5_Reverse, symbol Connector_Generic:Conn_02x05_Counter_Clockwise
- added J21: PERRI_21, HELIX:Perri_conn_2x5_Reverse, symbol Connector_Generic:Conn_02x05_Counter_Clockwise
- added J22: PERRI_22, HELIX:Perri_conn_2x5_Reverse, symbol Connector_Generic:Conn_02x05_Counter_Clockwise
- added J23: PERRI_23, HELIX:Perri_conn_2x5_Reverse, symbol Connector_Generic:Conn_02x05_Counter_Clockwise
- added J24: PERRI_24, HELIX:Perri_conn_2x5_Reverse, symbol Connector_Generic:Conn_02x05_Counter_Clockwise
- added J25: Probe 0, Connector_PinHeader_2.54mm:PinHeader_1x03_P2.54mm_Vertical, symbol Connector_Generic:Conn_01x03
- added J26: Probe 1, Connector_PinHeader_2.54mm:PinHeader_1x03_P2.54mm_Vertical, symbol Connector_Generic:Conn_01x03
- added J27: Probe 2, Connector_PinHeader_2.54mm:PinHeader_1x03_P2.54mm_Vertical, symbol Connector_Generic:Conn_01x03
- added J28: Probe 3, Connector_PinHeader_2.54mm:PinHeader_1x03_P2.54mm_Vertical, symbol Connector_Generic:Conn_01x03
- added J29: Power, Connector_Molex:Molex_Micro-Fit_3.0_43650-0400_1x04_P3.00mm_Horizontal, symbol Connector_Generic:Conn_01x04
- added J9: PERRI_9, HELIX:Perri_conn_2x5_Reverse, symbol Connector_Generic:Conn_02x05_Counter_Clockwise
- added R1, R2, R3, R4, R5, R6, R7, R8: Resistor, Resistor_SMD:R_0805_2012Metric, symbol Device:R_US
- added U1: EK-TM4C123GXL, HELIX:TM4C123GXL_launchpad_male_connector, symbol local:DEV_KIT_EK-TM4C123GXL
- H1, H2, H3, H4: value MountingHole_Pad -> Mount
Connections:
- net GND: now also H1.1, H2.1, H3.1, H4.1, J10.10 (Pin_10), J11.10 (Pin_10), J12.10 (Pin_10), J13.10 (Pin_10), J14.10 (Pin_10), J15.10 (Pin_10), J16.10 (Pin_10), J17.10 (Pin_10), J18.10 (Pin_10), J19.10 (Pin_10), J20.10 (Pin_10), J21.10 (Pin_10), J22.10 (Pin_10), J23.10 (Pin_10), J24.10 (Pin_10), J25.3 (Pin_3), J26.3 (Pin_3), J27.3 (Pin_3), J28.3 (Pin_3), J29.4 (Pin_4), J9.10 (Pin_10), U1.20 (GND), U1.22 (GND)
- net SCL renamed SCL_0
- net SCL_0: now also J25.1 (Pin_1), R2.1, U1.19 (PB2)
- net SDA renamed SDA_0
- net SDA_0: now also J25.2 (Pin_2), R1.1, U1.38 (PB3)
- new net +5V: J29.1 (Pin_1), R1.2, R2.2, R3.2, R4.2, R5.2, R6.2, R7.2, R8.2, U1.21 (5V)
- new net SCL_1: J10.5 (Pin_5), J11.5 (Pin_5), J12.5 (Pin_5), J13.5 (Pin_5), J14.5 (Pin_5), J15.5 (Pin_5), J16.5 (Pin_5), J26.1 (Pin_1), J9.5 (Pin_5), R4.1, U1.9 (PA6)
- new net SCL_2: J17.5 (Pin_5), J18.5 (Pin_5), J19.5 (Pin_5), J20.5 (Pin_5), J27.1 (Pin_1), R6.1, U1.5 (PE4)
- new net SCL_3: J21.5 (Pin_5), J22.5 (Pin_5), J23.5 (Pin_5), J24.5 (Pin_5), J28.1 (Pin_1), R8.1, U1.23 (PD0)
- new net SDA_1: J10.6 (Pin_6), J11.6 (Pin_6), J12.6 (Pin_6), J13.6 (Pin_6), J14.6 (Pin_6), J15.6 (Pin_6), J16.6 (Pin_6), J26.2 (Pin_2), J9.6 (Pin_6), R3.1, U1.10 (PA7)
- new net SDA_2: J17.6 (Pin_6), J18.6 (Pin_6), J19.6 (Pin_6), J20.6 (Pin_6), J27.2 (Pin_2), R5.1, U1.6 (PE5)
- new net SDA_3: J21.6 (Pin_6), J22.6 (Pin_6), J23.6 (Pin_6), J24.6 (Pin_6), J28.2 (Pin_2), R7.1, U1.24 (PD1)
- no-connect marks 56 -> 199
Other:
- note added: "I2C #1 SDA PA7 SCL PA8 I2C #2 SDA PE4 SCL PE5 I2C #3 SDA PD1 SCL PD0 I2C #4 SDA PB3 SCL PB2"
- note added: "Probe Points"
- note added: "Pull Up Resistors"
- company: (none) -> The Ohio State University
- title: (none) -> Perri_I2C_Breakout
- moved on the sheet: H1, H2, H3, H4
